Commit message: Adding lidar, camera and force torques.

File: src/go2_description/urdf/go2.urdf.xacro (robot description, xacro)
@@ -187,4 +187,28 @@
     <origin xyz="0 0 0" rpy="0 0 0"/>
   </joint>
+  <!-- LiDAR sensor link -->
+  <link name="lidar_link">
+    <visual>
+      <geometry><cylinder radius="0.03" length="0.04"/></geometry>
+      <material name="black"><color rgba="0.1 0.1 0.1 1.0"/></material>
+    </visual>
+  </link>
+  <joint name="lidar_joint" type="fixed">
+    <parent link="base_link"/>
+    <child  link="lidar_link"/>
+    <origin xyz="0.15 0 0.07" rpy="0 0 0"/>
+  </joint>
+  <!-- Camera sensor link -->
+  <link name="camera_link">
+    <visual>
+      <geometry><box size="0.02 0.05 0.02"/></geometry>
+      <material name="black"><color rgba="0.1 0.1 0.1 1.0"/></material>
+    </visual>
+  </link>
+  <joint name="camera_joint" type="fixed">
+    <parent link="base_link"/>
+    <child  link="camera_link"/>
+    <origin xyz="0.19 0 0.0" rpy="0 0 0"/>
+  </joint>
   <!-- ================================================================
        Legs (instantiate macro × 4)
@@ -248,6 +272,57 @@
     </sensor>
   </gazebo>
-  <!-- Foot contact sensors -->
-  <xacro:macro name="foot_contact_sensor" params="prefix">
+  <!-- LiDAR Gazebo sensor -->
+  <gazebo reference="lidar_link">
+    <sensor name="lidar" type="gpu_lidar">
+      <always_on>true</always_on>
+      <update_rate>10</update_rate>
+      <topic>/lidar/points</topic>
+      <gz_frame_id>lidar_link</gz_frame_id>
+      <lidar>
+        <scan>
+          <horizontal>
+            <samples>360</samples>
+            <resolution>1</resolution>
+            <min_angle>-3.14159</min_angle>
+            <max_angle>3.14159</max_angle>
+          </horizontal>
+          <vertical>
+            <samples>16</samples>
+            <resolution>1</resolution>
+            <min_angle>-0.26</min_angle>
+            <max_angle>0.26</max_angle>
+          </vertical>
+        </scan>
+        <range>
+          <min>0.1</min>
+          <max>30.0</max>
+          <resolution>0.01</resolution>
+        </range>
+      </lidar>
+    </sensor>
+  </gazebo>
+  <!-- Camera Gazebo sensor -->
+  <gazebo reference="camera_link">
+    <sensor name="camera" type="camera">
+      <always_on>true</always_on>
+      <update_rate>30</update_rate>
+      <topic>/camera/image_raw</topic>
+      <gz_frame_id>camera_link</gz_frame_id>
+      <camera>
+        <horizontal_fov>1.5</horizontal_fov>
+        <image>
+          <width>640</width>
+          <height>480</height>
+          <format>R8G8B8</format>
+        </image>
+        <clip>
+          <near>0.1</near>
+          <far>100</far>
+        </clip>
+      </camera>
+    </sensor>
+  </gazebo>
+  <!-- Foot sensors (contact + force/torque) -->
+  <xacro:macro name="foot_sensors" params="prefix">
     <gazebo reference="${prefix}_foot">
       <sensor name="${prefix}_foot_contact" type="contact">
@@ -258,8 +333,20 @@
       </sensor>
     </gazebo>
+    <gazebo reference="${prefix}_foot_fixed">
+      <preserveFixedJoint>true</preserveFixedJoint>
+      <sensor name="${prefix}_force_torque" type="force_torque">
+        <always_on>true</always_on>
+        <update_rate>100</update_rate>
+        <topic>/go2/${prefix}_force_torque</topic>
+        <force_torque>
+          <frame>child</frame>
+          <measure_direction>child_to_parent</measure_direction>
+        </force_torque>
+      </sensor>
+    </gazebo>
   </xacro:macro>
-  <xacro:foot_contact_sensor prefix="FL"/>
-  <xacro:foot_contact_sensor prefix="FR"/>
-  <xacro:foot_contact_sensor prefix="RL"/>
-  <xacro:foot_contact_sensor prefix="RR"/>
+  <xacro:foot_sensors prefix="FL"/>
+  <xacro:foot_sensors prefix="FR"/>
+  <xacro:foot_sensors prefix="RL"/>
+  <xacro:foot_sensors prefix="RR"/>
 </robot>

Commit message: Add go2 parts file paths.
Fix GPU use.

File: src/go2_description/urdf/go2.urdf.xacro (robot description, xacro)
@@ -72,6 +72,8 @@
     <link name="${prefix}_hip">
       <visual>
-        <geometry><cylinder radius="0.046" length="${hip_length}"/></geometry>
-        <origin xyz="0 ${reflect_y*hip_length/2} 0" rpy="${pi/2} 0 0"/>
+        <origin rpy="${(1-reflect_y)/2 * pi} ${(1-reflect_x)/2 * pi} 0" xyz="0 0 0"/>
+        <geometry>
+          <mesh filename="file://$(find go2_description)/meshes/hip.dae" scale="1 1 1"/>
+        </geometry>
       </visual>
       <collision>
@@ -94,6 +96,8 @@
     <link name="${prefix}_thigh">
       <visual>
-        <geometry><box size="0.05 0.04 ${thigh_length}"/></geometry>
-        <origin xyz="0 0 ${-thigh_length/2}" rpy="0 0 0"/>
+        <origin xyz="0 0 0" rpy="0 0 0"/>
+        <geometry>
+          <mesh filename="file://$(find go2_description)/meshes/thigh${'' if reflect_y == 1 else '_mirror'}.dae" scale="1 1 1"/>
+        </geometry>
       </visual>
       <collision>
@@ -116,6 +120,8 @@
     <link name="${prefix}_calf">
       <visual>
-        <geometry><box size="0.04 0.028 ${calf_length}"/></geometry>
-        <origin xyz="0 0 ${-calf_length/2}" rpy="0 0 0"/>
+        <origin xyz="0 0 0" rpy="0 0 0"/>
+        <geometry>
+          <mesh filename="file://$(find go2_description)/meshes/calf.dae" scale="1 1 1"/>
+        </geometry>
       </visual>
       <collision>
@@ -138,5 +144,8 @@
     <link name="${prefix}_foot">
       <visual>
-        <geometry><sphere radius="${foot_radius}"/></geometry>
+        <origin xyz="0 0 0" rpy="0 0 0"/>
+        <geometry>
+          <mesh filename="file://$(find go2_description)/meshes/foot.dae" scale="1 1 1"/>
+        </geometry>
       </visual>
       <collision>
@@ -163,10 +172,8 @@
   <link name="base_link">
     <visual>
+      <origin xyz="0 0 0" rpy="0 0 0"/>
       <geometry>
-        <box size="${body_length} ${body_width*2} ${body_height}"/>
+        <mesh filename="file://$(find go2_description)/meshes/base.dae" scale="1 1 1"/>
       </geometry>
-      <material name="dark_gray">
-        <color rgba="0.2 0.2 0.2 1.0"/>
-      </material>
     </visual>
     <collision>

Commit message: Add follow + apprehend mode.
Robot is able to detect and follow and intruder.
It has now a siren that is on when the intrudes is apprehended.

File: src/go2_description/urdf/go2.urdf.xacro (robot description, xacro)
@@ -91,5 +91,5 @@
       <limit lower="${-hip_limit}" upper="${hip_limit}"
              effort="${effort_limit}" velocity="${velocity_limit}"/>
-      <dynamics damping="0.1" friction="0.0"/>
+      <dynamics damping="3.0" friction="0.2"/>
     </joint>
     <!-- Thigh link -->
@@ -115,5 +115,5 @@
       <limit lower="${thigh_lower}" upper="${thigh_upper}"
              effort="${effort_limit}" velocity="${velocity_limit}"/>
-      <dynamics damping="0.1" friction="0.0"/>
+      <dynamics damping="3.0" friction="0.2"/>
     </joint>
     <!-- Calf link -->
@@ -139,5 +139,5 @@
       <limit lower="${calf_lower}" upper="${calf_upper}"
              effort="${effort_limit}" velocity="${velocity_limit}"/>
-      <dynamics damping="0.1" friction="0.0"/>
+      <dynamics damping="3.0" friction="0.2"/>
     </joint>
     <!-- Foot (sphere — for contact) -->
@@ -152,5 +152,5 @@
         <geometry><sphere radius="${foot_radius}"/></geometry>
         <surface>
-          <friction><ode><mu>0.8</mu><mu2>0.8</mu2></ode></friction>
+          <friction><ode><mu>1.5</mu><mu2>1.5</mu2></ode></friction>
         </surface>
       </collision>
@@ -309,4 +309,26 @@
     </sensor>
   </gazebo>
+  <!-- Siren light mount -->
+  <link name="siren_link">
+    <visual name="siren_light">
+      <origin xyz="0 0 0.015" rpy="0 0 0"/>
+      <geometry><cylinder radius="0.025" length="0.03"/></geometry>
+      <material name="siren_red"><color rgba="0.9 0.1 0.1 0.9"/></material>
+    </visual>
+    <visual name="siren_base">
+      <origin xyz="0 0 0.0" rpy="0 0 0"/>
+      <geometry><cylinder radius="0.03" length="0.015"/></geometry>
+      <material name="siren_base_mat"><color rgba="0.2 0.2 0.2 1.0"/></material>
+    </visual>
+    <inertial>
+      <mass value="0.05"/>
+      <inertia ixx="0.00001" ixy="0" ixz="0" iyy="0.00001" iyz="0" izz="0.00001"/>
+    </inertial>
+  </link>
+  <joint name="siren_joint" type="fixed">
+    <parent link="base_link"/>
+    <child  link="siren_link"/>
+    <origin xyz="-0.05 0 0.08" rpy="0 0 0"/>
+  </joint>
   <!-- Camera Gazebo sensor -->
   <gazebo reference="camera_link">
